File: eletric.brd (EAGLE design)
At the start: 69.4 x 118.6 mm, 15 parts, among them U1 ATTINY85-20PU

Commit message: center piezos (clothing button)
Parts:
- moved LS3 9.53 mm to (50.2, 55.9)
- moved LS2 5.71 mm to (50.2, 17.1)
- moved LS4 1.27 mm to (50.2, 29.8)
Routing:
- net N$4: track 47.2 -> 37.7 mm
- net BUZER_HARMONY_3: track 63.0 -> 54.3 mm
- net BUZER_HARMONY_2: track 82.9 -> 88.7 mm
- net N$3: track 88.6 -> 82.9 mm
- net BUZER_HARMONY_1: track 102.2 -> 103.6 mm
- net N$2: track 66.1 -> 65.3 mm
